File: KiCad/edu-80/Protected RAM.kicad_sch (KiCad schematic)
At the start: 8 parts, among them U24 2111A, U25 2111A, U26 2111A, U27 2111A, U28 2111A, U29 2111A, U30 2111A, U31 2111A

Commit message: Working on removing edu-80-rescue symbol library
Parts:
- removed U28, U29, U31: 2111A, Package_DIP:DIP-20_W7.62mm, symbol edu-80-rescue:2111A-Edu-80_Symbol
- added U28, U29, U31: 2111A, Package_DIP:DIP-20_W7.62mm, symbol Edu-80_Symbols:2111A
- U30: symbol edu-80-rescue:2111A-Edu-80_Symbol -> Edu-80_Symbols:2111A
Connections:
- net +5V: now also U28.18 (VCC), U29.18 (VCC), U31.18 (VCC)
- net A0: now also U28.17 (A4), U29.17 (A4), U31.17 (A4)
- net A1: now also U28.7 (A7), U29.7 (A7), U31.7 (A7)
- net A2: now also U28.6 (A6), U29.6 (A6), U31.6 (A6)
- net A3: now also U28.5 (A5), U29.5 (A5), U31.5 (A5)
- net A4: now also U28.4 (A0), U29.4 (A0), U31.4 (A0)
- net A5: now also U28.3 (A1), U29.3 (A1), U31.3 (A1)
- net A6: now also U28.2 (A2), U29.2 (A2), U31.2 (A2)
- net A7: now also U28.1 (A3), U29.1 (A3), U31.1 (A3)
- net CM1: now also U28.15 (~{CE2}), U29.15 (~{CE2}), U31.15 (~{CE2})
- net D0: now also U28.13 (D3)
- net D1: now also U28.12 (D2)
- net D2: now also U28.11 (D1)
- net D3: now also U28.14 (D4)
- net D4: now also U29.14 (D4), U31.14 (D4)
- net D5: now also U29.13 (D3), U31.13 (D3)
- net D6: now also U29.12 (D2), U31.12 (D2)
- net D7: now also U29.11 (D1), U31.11 (D1)
- net Earth: now also U28.8 (GND), U29.8 (GND), U31.8 (GND)
- net MRP: now also U28.16 (R/W), U29.16 (R/W), U31.16 (R/W)
- net ~{ME3}: now also U28.10 (~{CE1}), U29.10 (~{CE1})
- net ~{ME4}: now also U31.10 (~{CE1})
- net ~{RD}: now also U28.9 (~{OE}), U29.9 (~{OE}), U31.9 (~{OE})

Commit message: Cleaning up the PAL-003 decoding, adding Modifications page.
Parts:
- U24, U25, U26, U27: symbol edu-80-rescue:2111A-Edu-80_Symbol -> Edu-80_Symbols:2111A
Changed lines of the file:
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@@
   (title_block
     (title "Edu-80 Z80 Trainer")
-    (date "2023-02-06")
+    (date "2023-06-03")
     (rev "0.1")
     (company "Strangers")
+    (comment 1 "Author: James D. Tucker")
   )
   (junction (at 196.85 25.4) (diameter 0) (color 0 0 0 0)
@@
     )
   )
-  (symbol (lib_id "edu-80-rescue:2111A-Edu-80_Symbol") (at 60.96 114.3 0) (unit 1)
+  (symbol (lib_id "Edu-80_Symbols:2111A") (at 60.96 114.3 0) (unit 1)
     (in_bom yes) (on_board yes) (dnp no)
     (property "Reference" "U24" (at 60.96 96.139 0)
@@
     )
   )
-  (symbol (lib_id "edu-80-rescue:2111A-Edu-80_Symbol") (at 111.76 55.88 0) (unit 1)
+  (symbol (lib_id "Edu-80_Symbols:2111A") (at 111.76 55.88 0) (unit 1)
     (in_bom yes) (on_board yes) (dnp no)
     (property "Reference" "U27" (at 111.76 37.719 0)
@@
     )
   )
-  (symbol (lib_id "edu-80-rescue:2111A-Edu-80_Symbol") (at 60.96 55.88 0) (unit 1)
+  (symbol (lib_id "Edu-80_Symbols:2111A") (at 60.96 55.88 0) (unit 1)
     (in_bom yes) (on_board yes) (dnp no)
     (property "Reference" "U25" (at 60.96 37.719 0)
@@
     )
   )
-  (symbol (lib_id "edu-80-rescue:2111A-Edu-80_Symbol") (at 111.76 114.3 0) (unit 1)
+  (symbol (lib_id "Edu-80_Symbols:2111A") (at 111.76 114.3 0) (unit 1)
     (in_bom yes) (on_board yes) (dnp no)
     (property "Reference" "U26" (at 111.76 96.139 0)

Commit message: Fixed the last of the EDR warnings/errors, adding footprints
Parts:
- U24, U25, U26, U27, U28, U29, U30, U31: footprint Package_DIP:DIP-20_W7.62mm -> Package_DIP:DIP-18_W7.62mm
Changed lines of the file:
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@@
       (effects (font (size 1.27 1.27)))
     )
-    (property "Footprint" "Package_DIP:DIP-20_W7.62mm" (at 60.96 100.33 0)
+    (property "Footprint" "Package_DIP:DIP-18_W7.62mm" (at 60.96 100.33 0)
       (effects (font (size 1.27 1.27)) hide)
     )
@@
       (effects (font (size 1.27 1.27)))
     )
-    (property "Footprint" "Package_DIP:DIP-20_W7.62mm" (at 160.02 100.33 0)
+    (property "Footprint" "Package_DIP:DIP-18_W7.62mm" (at 160.02 100.33 0)
       (effects (font (size 1.27 1.27)) hide)
     )
@@
       (effects (font (size 1.27 1.27)))
     )
-    (property "Footprint" "Package_DIP:DIP-20_W7.62mm" (at 210.82 100.33 0)
+    (property "Footprint" "Package_DIP:DIP-18_W7.62mm" (at 210.82 100.33 0)
       (effects (font (size 1.27 1.27)) hide)
     )
@@
       (effects (font (size 1.27 1.27)))
     )
-    (property "Footprint" "Package_DIP:DIP-20_W7.62mm" (at 111.76 41.91 0)
+    (property "Footprint" "Package_DIP:DIP-18_W7.62mm" (at 111.76 41.91 0)
       (effects (font (size 1.27 1.27)) hide)
     )
@@
       (effects (font (size 1.27 1.27)))
     )
-    (property "Footprint" "Package_DIP:DIP-20_W7.62mm" (at 210.82 41.91 0)
+    (property "Footprint" "Package_DIP:DIP-18_W7.62mm" (at 210.82 41.91 0)
       (effects (font (size 1.27 1.27)) hide)
     )
@@
       (effects (font (size 1.27 1.27)))
     )
-    (property "Footprint" "Package_DIP:DIP-20_W7.62mm" (at 60.96 41.91 0)
+    (property "Footprint" "Package_DIP:DIP-18_W7.62mm" (at 60.96 41.91 0)
       (effects (font (size 1.27 1.27)) hide)
     )
@@
       (effects (font (size 1.27 1.27)))
     )
-    (property "Footprint" "Package_DIP:DIP-20_W7.62mm" (at 111.76 100.33 0)
+    (property "Footprint" "Package_DIP:DIP-18_W7.62mm" (at 111.76 100.33 0)
       (effects (font (size 1.27 1.27)) hide)
     )
@@
       (effects (font (size 1.27 1.27)))
     )
-    (property "Footprint" "Package_DIP:DIP-20_W7.62mm" (at 160.02 41.91 0)
-      (effects (font (size 1.27 1.27)) hide)
-    )
+    (property "Footprint" "Package_DIP:DIP-18_W7.62mm" (at 160.02 41.91 0)
+      (effects (font (size 1.27 1.27)) hide)
+    )
