File: KiCad/edu-80/BreadBoard.kicad_sch (KiCad schematic)
At the start: 5 parts

Commit message: Adding footprints.
Parts:
- S1, S2, S3, S4, S5: footprint (none) -> Connector_PinSocket_1.00mm:PinSocket_1x16_P1.00mm_Vertical
Changed lines of the file:
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@@
       (effects (font (size 1.27 1.27)) (justify left))
     )
-    (property "Footprint" "" (at 62.23 87.63 0)
+    (property "Footprint" "Connector_PinSocket_1.00mm:PinSocket_1x16_P1.00mm_Vertical" (at 62.23 87.63 0)
       (effects (font (size 1.27 1.27)) hide)
     )
@@
       (effects (font (size 1.27 1.27)) (justify left))
     )
-    (property "Footprint" "" (at 100.33 87.63 0)
+    (property "Footprint" "Connector_PinSocket_1.00mm:PinSocket_1x16_P1.00mm_Vertical" (at 100.33 87.63 0)
       (effects (font (size 1.27 1.27)) hide)
     )
@@
       (effects (font (size 1.27 1.27)) (justify left))
     )
-    (property "Footprint" "" (at 138.43 87.63 0)
+    (property "Footprint" "Connector_PinSocket_1.00mm:PinSocket_1x16_P1.00mm_Vertical" (at 138.43 87.63 0)
       (effects (font (size 1.27 1.27)) hide)
     )
@@
       (effects (font (size 1.27 1.27)) (justify left))
     )
-    (property "Footprint" "" (at 176.53 87.63 0)
+    (property "Footprint" "Connector_PinSocket_1.00mm:PinSocket_1x16_P1.00mm_Vertical" (at 176.53 87.63 0)
       (effects (font (size 1.27 1.27)) hide)
     )
@@
       (effects (font (size 1.27 1.27)) (justify left))
     )
-    (property "Footprint" "" (at 214.63 87.63 0)
+    (property "Footprint" "Connector_PinSocket_1.00mm:PinSocket_1x16_P1.00mm_Vertical" (at 214.63 87.63 0)
       (effects (font (size 1.27 1.27)) hide)
     )
