File: KiCad/edu-80/PIO-CTC.kicad_sch (KiCad schematic)
At the start: 2 parts, among them U2 Z84C20, U3 Z8430_CTC

Commit message: Adding footprints.
Parts:
- added U4: Z80-CTC, Package_DIP:DIP-28_W15.24mm_Socket, symbol jb-symbol:Z80_CTC
Changed lines of the file:
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@@
+    )
+  )
+  (symbol (lib_id "jb-symbol:Z80_CTC") (at 236.22 137.16 0) (mirror y) (unit 1)
+    (in_bom yes) (on_board yes) (dnp no)
+    (property "Reference" "U4" (at 227.33 109.22 0)
+      (effects (font (size 1.27 1.27)))
+    )
+    (property "Value" "Z80-CTC" (at 226.06 111.76 0)
+      (effects (font (size 1.27 1.27)))
+    )
+    (property "Footprint" "Package_DIP:DIP-28_W15.24mm_Socket" (at 210.82 105.41 0)
+      (effects (font (size 1.27 1.27)) hide)
+    )
+    (property "Datasheet" "http://www.zilog.com/docs/z80/ps0181.pdf" (at 236.22 137.16 0)
+      (effects (font (size 1.27 1.27)) hide)
+    )
+    (property "Digi-Key_PN" "269-3914-ND" (at 236.22 137.16 0)
+      (effects (font (size 1.27 1.27)) hide)
+    )
+    (property "MPN" "Z84C3010PEG‎" (at 236.22 137.16 0)
+      (effects (font (size 1.27 1.27)) hide)
+    )
+    (property "Description" "IC Z80 CTC 10MHZ 28DIP" (at 236.22 137.16 0)
+      (effects (font (size 1.27 1.27)) hide)
+    )
+    (property "Manufacturer" "Zilog" (at 236.22 137.16 0)
+      (effects (font (size 1.27 1.27)) hide)
+    )
+    (pin "24")
+    (pin "5")
+    (pin "1")
+    (pin "10")
+    (pin "11")
+    (pin "12")
+    (pin "13")
+    (pin "14")
+    (pin "15")
+    (pin "16")
+    (pin "17")
+    (pin "18")
+    (pin "19")
+    (pin "2")
+    (pin "20")
+    (pin "21")
+    (pin "22")
+    (pin "23")
+    (pin "25")
+    (pin "26")
+    (pin "27")
+    (pin "28")
+    (pin "3")
+    (pin "4")
+    (pin "6")
+    (pin "7")
+    (pin "8")
+    (pin "9")
+    (instances
+      (project "2063-Z80"
+        (path "/5c376030-5ec1-4a75-bca4-de6cdb0fa1a8"
+          (reference "U4") (unit 1)
+        )
+      )
+      (project "edu-80"
+        (path "/d19d6db6-a96a-43e3-aa50-c057821f7e22/00000000-0000-0000-0000-00006442bb97"
+          (reference "U40") (unit 1)
+        )
+      )
     )
   )
