File: KiCad/edu-80/edu-80.kicad_pcb (KiCad board)
At the start: 2 copper layers, 111 parts, among them Q1 ED1402, Q10 ED1602, Q11 ED1602, Q12 ED1602, Q13 ED1602, Q14 ED1602, Q15 ED1602, Q16 ED1602, Q17 ED1602, Q18 ED1602, Q19 ED1602, Q2 ED1402, Q20 ED1602, Q21 2N3055, Q22 2N3906, Q3 ED1402, Q4 ED1602, Q5 ED1602, Q6 ED1602, Q7 ED1602, Q8 ED1602, Q9 ED1602, U10 7442, U101 7408, U14 PAL-002, U17 PAL-001, U18 CD4051, U19 CD4099, U2 Z84C20, U20 CD4099, U21 7442, U24 2111A, U25 2111A, U26 2111A, U27 2111A, U28 2111A, U29 2111A, U3 Z8430_CTC, U30 2111A, U31 2111A, U32 2111A, U33 2111A, U34 2111A, U35 2111A, U36 2111A, U37 2111A, U38 2111A, U39 2111A, U4 EPROM-2708, U5 2708_(2716), U6 6116_RAM, U7 EPROM-2708, U8 SN7432, U9 7442, X1 20MHz Ocillator

Commit message: Adding footprints.
Parts:
- added C1: 20p, Capacitor_THT:CP_Radial_D5.0mm_P2.00mm, F.Cu at (78.5, 3.01)
- added C10: 1000 uF (16v), Capacitor_THT:CP_Radial_D10.0mm_P2.50mm_P5.00mm, F.Cu at (1.48, 5.28)
- added C11: 100 uF (16v), Capacitor_THT:CP_Radial_D10.0mm_P2.50mm_P5.00mm, F.Cu at (1.48, 16.8)
- added C12: 2200 uF (16v), Capacitor_THT:CP_Radial_D10.0mm_P2.50mm_P5.00mm, F.Cu at (1.48, 28.4)
- added C13: 1000 uF (16v), Capacitor_THT:CP_Radial_D10.0mm_P2.50mm_P5.00mm, F.Cu at (1.48, 39.9)
- added C2: 10p, Capacitor_THT:CP_Radial_D5.0mm_P2.00mm, F.Cu at (78.5, 9.54)
- added C3: 250p, Capacitor_THT:CP_Radial_D5.0mm_P2.00mm, F.Cu at (78.5, 16.1)
- added D6: D_Bridge_+-AA, Diode_THT:Diode_Bridge_15.1x15.1x6.3mm_P10.9mm, F.Cu at (32.3, 2.38)
- added J1: Audio Out, Connector_Audio:Jack_3.5mm_CUI_SJ-3523-SMT_Horizontal, F.Cu at (54.3, 82.3)
- added J2: Audio In, Connector_Audio:Jack_3.5mm_CUI_SJ-3523-SMT_Horizontal, F.Cu at (66.5, 82.3)
- added J3: Conn_01x03, Connector:FanPinHeader_1x03_P2.54mm_Vertical, F.Cu at (79.0, 22.7)
- added JP1: SolderJumper_2_Open, Jumper:SolderJumper-2_P1.3mm_Open_RoundedPad1.0x1.5mm, F.Cu at (80.9, 55.5)
- added JP2: SolderJumper_2_Open, Jumper:SolderJumper-2_P1.3mm_Open_RoundedPad1.0x1.5mm, F.Cu at (80.9, 59.1)
- added JP3: SolderJumper_2_Open, Jumper:SolderJumper-2_P1.3mm_Open_RoundedPad1.0x1.5mm, F.Cu at (80.9, 62.6)
- added JP4: SolderJumper_2_Open, Jumper:SolderJumper-2_P1.3mm_Open_RoundedPad1.0x1.5mm, F.Cu at (80.9, 66.2)
- added JP5: SolderJumper_2_Open, Jumper:SolderJumper-2_P1.3mm_Open_RoundedPad1.0x1.5mm, F.Cu at (80.9, 69.7)
- added R1: 330, Resistor_THT:R_Axial_DIN0309_L9.0mm_D3.2mm_P25.40mm_Horizontal, F.Cu at (49.7, 1.88)
- added R11: 4.7K, Resistor_THT:R_Axial_DIN0309_L9.0mm_D3.2mm_P25.40mm_Horizontal, F.Cu at (49.7, 35.1)
- added R12: 4.7K, Resistor_THT:R_Axial_DIN0309_L9.0mm_D3.2mm_P25.40mm_Horizontal, F.Cu at (49.7, 39.9)
- added R13: 4.7K, Resistor_THT:R_Axial_DIN0309_L9.0mm_D3.2mm_P25.40mm_Horizontal, F.Cu at (49.7, 44.6)
- added R14: 4.7K, Resistor_THT:R_Axial_DIN0309_L9.0mm_D3.2mm_P25.40mm_Horizontal, F.Cu at (49.7, 49.4)
- added R15: 330, Resistor_THT:R_Axial_DIN0309_L9.0mm_D3.2mm_P25.40mm_Horizontal, F.Cu at (49.7, 56.1)
- added R16: 10K, Resistor_THT:R_Axial_DIN0309_L9.0mm_D3.2mm_P25.40mm_Horizontal, F.Cu at (49.7, 60.9)
- added R17: 10K, Resistor_THT:R_Axial_DIN0309_L9.0mm_D3.2mm_P25.40mm_Horizontal, F.Cu at (49.7, 65.6)
- added R18: 1K, Resistor_THT:R_Axial_DIN0309_L9.0mm_D3.2mm_P25.40mm_Horizontal, F.Cu at (49.7, 70.4)
- added R2: 4.7K, Resistor_THT:R_Axial_DIN0309_L9.0mm_D3.2mm_P25.40mm_Horizontal, F.Cu at (49.7, 6.62)
- added R3: 1M, Resistor_THT:R_Axial_DIN0309_L9.0mm_D3.2mm_P25.40mm_Horizontal, F.Cu at (49.7, 11.4)
- added R4: 10K, Resistor_THT:R_Axial_DIN0309_L9.0mm_D3.2mm_P25.40mm_Horizontal, F.Cu at (49.7, 16.1)
- added R5: 10K, Resistor_THT:R_Axial_DIN0309_L9.0mm_D3.2mm_P25.40mm_Horizontal, F.Cu at (49.7, 20.9)
- added R6: 30K, Resistor_THT:R_Axial_DIN0309_L9.0mm_D3.2mm_P25.40mm_Horizontal, F.Cu at (49.7, 25.6)
- added R7: 100K, Resistor_THT:R_Axial_DIN0309_L9.0mm_D3.2mm_P25.40mm_Horizontal, F.Cu at (49.7, 30.4)
- added R8: 470, Resistor_THT:R_Axial_DIN0309_L9.0mm_D3.2mm_P25.40mm_Horizontal, F.Cu at (1.07, 48.1)
- added R9: 470, Resistor_THT:R_Axial_DIN0309_L9.0mm_D3.2mm_P25.40mm_Horizontal, F.Cu at (1.07, 52.8)
- C4, C5, C6, C7, C8, C9: footprint Capacitor_THT:CP_Radial_D5.0mm_P2.50mm -> Capacitor_THT:CP_Radial_D5.0mm_P2.00mm
